Commit message: Hastane koridoru dünyası, tek launch dosyası ve ok tuşlu sürüş eklendi

File: ros2_ws/src/lokman_description/urdf/chassis.xacro (robot description, xacro)
@@ -45,5 +45,5 @@
       <origin xyz="${kasa_arka_x + kasa_l/2} 0 ${sasi_z}"/>
       <geometry><box size="${kasa_l} ${govde_w} ${sasi_h}"/></geometry>
-      <material name="hastane_beyazi"/>
+      <xacro:renk ad="hastane_beyazi"/>
     </visual>
     <collision>
@@ -55,5 +55,5 @@
       <origin xyz="${burun_x} 0 ${sasi_z}"/>
       <geometry><cylinder radius="${burun_r}" length="${sasi_h}"/></geometry>
-      <material name="hastane_beyazi"/>
+      <xacro:renk ad="hastane_beyazi"/>
     </visual>
     <collision>
@@ -65,10 +65,10 @@
       <origin xyz="${kasa_arka_x + kasa_l/2} 0 0.12"/>
       <geometry><box size="${kasa_l + 0.004} ${govde_w + 0.004} 0.035"/></geometry>
-      <material name="turkuaz"/>
+      <xacro:renk ad="turkuaz"/>
     </visual>
     <visual>
       <origin xyz="${burun_x} 0 0.12"/>
       <geometry><cylinder radius="${burun_r + 0.002}" length="0.035"/></geometry>
-      <material name="turkuaz"/>
+      <xacro:renk ad="turkuaz"/>
     </visual>
     <!-- Kütle: bataryalar tabanda → 18 kg, ağırlık merkezi alçakta -->
@@ -79,5 +79,5 @@
     <visual>
       <geometry><box size="${kabin_l} ${kabin_w} ${kabin_h}"/></geometry>
-      <material name="kabin_grisi"/>
+      <xacro:renk ad="kabin_grisi"/>
     </visual>
     <collision>
@@ -90,20 +90,20 @@
       <origin xyz="${-kabin_l/2 - 0.005} 0 0.14"/>
       <geometry><box size="0.01 ${kabin_w - 0.06} 0.24"/></geometry>
-      <material name="hastane_beyazi"/>
+      <xacro:renk ad="hastane_beyazi"/>
     </visual>
     <visual>
       <origin xyz="${-kabin_l/2 - 0.005} 0 -0.14"/>
       <geometry><box size="0.01 ${kabin_w - 0.06} 0.24"/></geometry>
-      <material name="hastane_beyazi"/>
+      <xacro:renk ad="hastane_beyazi"/>
     </visual>
     <visual>
       <origin xyz="${-kabin_l/2 - 0.02} 0 0.20"/>
       <geometry><box size="0.02 0.16 0.02"/></geometry>
-      <material name="metal"/>
+      <xacro:renk ad="metal"/>
     </visual>
     <visual>
       <origin xyz="${-kabin_l/2 - 0.02} 0 -0.08"/>
       <geometry><box size="0.02 0.16 0.02"/></geometry>
-      <material name="metal"/>
+      <xacro:renk ad="metal"/>
     </visual>
     <!-- Üstte turkuaz kapak ve yeşil durum feneri -->
@@ -111,10 +111,10 @@
       <origin xyz="0 0 ${kabin_h/2 + 0.01}"/>
       <geometry><box size="${kabin_l + 0.01} ${kabin_w + 0.01} 0.02"/></geometry>
-      <material name="turkuaz"/>
+      <xacro:renk ad="turkuaz"/>
     </visual>
     <visual>
       <origin xyz="0 0 ${kabin_h/2 + 0.04}"/>
       <geometry><cylinder radius="0.05" length="0.04"/></geometry>
-      <material name="durum_yesili"/>
+      <xacro:renk ad="durum_yesili"/>
     </visual>
     <xacro:kutu_inertia m="6.0" x="${kabin_l}" y="${kabin_w}" z="${kabin_h}"/>
@@ -134,5 +134,5 @@
         <origin rpy="${pi/2} 0 0"/>
         <geometry><cylinder radius="${teker_r}" length="${teker_w}"/></geometry>
-        <material name="koyu_gri"/>
+        <xacro:renk ad="koyu_gri"/>
       </visual>
       <!-- Jant göbeği: tekerleğin döndüğünü görebilmek için merkez dışı küçük bir işaret -->
@@ -140,5 +140,5 @@
         <origin xyz="0.035 ${y_isaret*teker_w/2} 0" rpy="${pi/2} 0 0"/>
         <geometry><cylinder radius="0.015" length="0.004"/></geometry>
-        <material name="turkuaz"/>
+        <xacro:renk ad="turkuaz"/>
       </visual>
       <collision>
@@ -172,5 +172,5 @@
       <visual>
         <geometry><sphere radius="${caster_r}"/></geometry>
-        <material name="metal"/>
+        <xacro:renk ad="metal"/>
       </visual>
       <collision>

File: ros2_ws/src/lokman_description/urdf/ortak.xacro (robot description, xacro)
@@ -7,12 +7,20 @@
 -->
 <robot xmlns:xacro="http://www.ros.org/wiki/xacro">
-  <!-- ===== Renk paleti (gerekçeler docs/tasarim.md, bölüm 4) ===== -->
-  <material name="hastane_beyazi"><color rgba="0.95 0.96 0.97 1"/></material>
-  <material name="turkuaz"><color rgba="0.0 0.65 0.65 1"/></material>
-  <material name="kabin_grisi"><color rgba="0.82 0.85 0.88 1"/></material>
-  <material name="koyu_gri"><color rgba="0.15 0.15 0.17 1"/></material>
-  <material name="metal"><color rgba="0.6 0.62 0.65 1"/></material>
-  <material name="durum_yesili"><color rgba="0.1 0.9 0.3 1"/></material>
-  <material name="bumper_turuncu"><color rgba="1.0 0.45 0.0 1"/></material>
+  <!-- ===== Renk paleti (gerekçeler docs/tasarim.md, bölüm 4) =====
+       Renkler her görsel parçanın İÇİNE yazılıyor (xacro:renk makrosu).
+       Dosyanın başında bir kez tanımlayıp adıyla çağırmak RViz'de renklerin
+       kaybolmasına (robotun gri görünmesine) yol açıyordu. -->
+  <xacro:property name="renkler" value="${dict(
+      hastane_beyazi = '0.95 0.96 0.97 1',
+      turkuaz        = '0.0 0.65 0.65 1',
+      kabin_grisi    = '0.82 0.85 0.88 1',
+      koyu_gri       = '0.15 0.15 0.17 1',
+      metal          = '0.6 0.62 0.65 1',
+      durum_yesili   = '0.1 0.9 0.3 1',
+      bumper_turuncu = '1.0 0.45 0.0 1')}"/>
+  <!-- Kullanım: <xacro:renk ad="turkuaz"/> -->
+  <xacro:macro name="renk" params="ad">
+    <material name="${ad}"><color rgba="${renkler[ad]}"/></material>
+  </xacro:macro>
   <!-- ===== Eylemsizlik makroları ===== -->
   <xacro:macro name="kutu_inertia" params="m x y z">
